File: PCB/Keypad_module.kicad_sch (KiCad schematic)
At the start: 72 parts, among them SW83 SW_Push, SW84 SW_Push, SW85 SW_Push, SW86 SW_Push, SW87 SW_Push, SW88 SW_Push, SW89 SW_Push, SW90 SW_Push, SW91 SW_Push, SW92 SW_Push, SW93 SW_Push, SW94 SW_Push, SW95 SW_Push, SW96 SW_Push, SW97 SW_Push, SW98 SW_Push, SW99 SW_Push, U5 XIAO-nRF52840-SMD, U6 MCP23017_ML, U8 74LV1T08GV

Commit message: Update README.md
Parts:
- Conn5, Conn6, Conn7, Conn8: Name (none) -> Connectors
- LED83, LED84, LED85, LED86, LED87, LED88, LED89, LED90, LED91, LED92, LED93, LED94, LED95, LED96, LED97, LED98, LED99: Name (none) -> LEDs
- RE1: Name (none) -> Rotary Encoder
- U8: Name (none) -> 74LV1T08GV
